File: Mixer.kicad_sch (KiCad schematic)
At the start: 48 parts, among them J1 Eurorack 2x8hs, J13 OUT1, J17 IN1, J18 IN2, J19 IN3, J20 IN4, J21 IN5, U1 TL072, U2 LM3915N

Commit message: Update to reduce FP traces and final self-etch print.
Parts:
- R11: footprint Resistor_THT:R_Axial_DIN0204_L3.6mm_D1.6mm_P2.54mm_Vertical -> Resistor_THT:R_Axial_DIN0204_L3.6mm_D1.6mm_P5.08mm_Horizontal
Changed lines of the file:
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@@
 			)
 		)
-		(property "Footprint" "Resistor_THT:R_Axial_DIN0204_L3.6mm_D1.6mm_P2.54mm_Vertical"
+		(property "Footprint" "Resistor_THT:R_Axial_DIN0204_L3.6mm_D1.6mm_P5.08mm_Horizontal"
 			(at 218.44 42.418 90)
 			(hide yes)
